File: Front Plate/Nearfield RP2040 FP.kicad_pcb (KiCad board)
At the start: 2 copper layers, 364.8 x 149.2 mm, 77 parts

Commit message: V1.00
Full design ready
Parts:
- added Logo1: CC-BY-SA-4.0, Logotypes:CC_BY_SA_40, B.Cu at (169.7, 185.3)
- H1, H2, H3, H4, H5, H6, H7, H8: footprint Keyboard_Plate:Spacer Plate hole -> Keyboard_Plate:Spacer_Plate_Grounded; moved to B.Cu
- ST1: footprint Keyboard_Plate:Stabilizer_Cherry_MX_2.00u_PLate_1_2 -> Keyboard_Plate:Stabilizer_Plate_2_to_1
- SW1, SW10, SW11, SW12, SW13, SW14, SW15, SW16, SW17, SW18, SW19, SW2, SW20, SW21, SW22, SW23, SW24, SW25, SW26, SW27, SW3, SW30, SW31, SW32, SW33, SW34, SW35, SW36, SW37, SW38, SW39, SW4, SW40, SW41, SW42, SW43, SW44, SW46, SW47, SW48, SW49, SW5, SW50, SW51, SW52, SW53, SW54, SW55, SW56, SW57, SW58, SW59, SW6, SW60, SW61, SW62, SW63, SW68, SW69, SW7, SW70, SW71, SW72, SW8, SW9: footprint Keyboard_Plate:SW_MX_Plate_Placeholder_nodrill_NOBORDER_13,9 -> Keyboard_Plate:SW_MX_Plate_Placeholder_nodrill
- turned H1 to 180 degrees
- turned H2 to 180 degrees
- turned H3 to 180 degrees
- turned H4 to 180 degrees
- turned H5 to 180 degrees
- turned H6 to 180 degrees
- turned H7 to 180 degrees
- turned H8 to 180 degrees
Routing:
- added copper zone on B.Cu, net GND
- added copper zone on F.Cu, net GND
- removed copper zone on B.Cu, net (none)
- removed copper zone on F.Cu, net (none)
Other:
- board size 364.8 x 149.2 mm -> 364.8 x 148.8 mm
- board text added: "JLCJLCJLCJLC"
- board text added: "Royal Enfield Plate - v1.00 Markus Knutsson 2024 https://github.com/TweetyDaBird"
