File: Front Plate/Nearfield RP2040 FP.kicad_sch (KiCad schematic)
At the start: 77 parts

Commit message: V1.00
Full design ready
Parts:
- added Logo1: CC-BY-SA-4.0, Logotypes:CC_BY_SA_40, symbol Logotypes:CC-BY-SA-4.0
- H1, H10, H2, H3, H6, H7, H8, H9: footprint Keyboard_Plate:Spacer Plate hole -> Keyboard_Plate:Spacer_Plate_Grounded; symbol Keyboard_Plate:Spacer_PCB -> Keyboard_Plate:Spacer_Plate_Grounded; now fitted
- ST1: footprint Keyboard_Plate:Stabilizer_Cherry_MX_2.00u_PLate_1_2 -> Keyboard_Plate:Stabilizer_Plate_2_to_1; now fitted
- SW10, SW11, SW13, SW14, SW15, SW16, SW17, SW18, SW19, SW2, SW20, SW21, SW22, SW23, SW24, SW26, SW27, SW28, SW29, SW3, SW30, SW31, SW32, SW33, SW34, SW35, SW39, SW4, SW45, SW5, SW6, SW7, SW8, SW9: footprint Keyboard_Plate:SW_MX_Plate_Placeholder_nodrill_NOBORDER_13,9 -> Keyboard_Plate:SW_MX_Plate_Placeholder_nodrill
Connections:
- new net GND: H1.1, H10.1, H2.1, H3.1, H6.1, H7.1, H8.1, H9.1
