File: PCB/Nearfield RP2040.kicad_sch (KiCad schematic)
At the start: 208 parts, among them J2 Conn_01x04, SW67 YTSA010, SW68 YTSA010, U2 W25Q32JVUUIQ, U3 RP2040, U3 SPX3819M5-L-3-3/TR, U4 SN74LV1T34DBV, Y1 TXM12M0004252LBCEO00T

Commit message: V1.00
Full design ready
Parts:
- J2: LCSC (none) -> C588524
Other:
- company: (none) -> Tweety's Wild Thinking
- title: (none) -> Royal Nearfield PCB
Changed lines of the file:
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@@
 (kicad_sch (version 20230121) (generator eeschema)
   (paper "A3")
+  (title_block
+    (title "Royal Nearfield PCB")
+    (date "2024-01-07")
+    (rev "v1.00")
+    (company "Tweety's Wild Thinking")
+    (comment 1 "Markus Knutsson <markus.knutsson@tweety.se>")
+    (comment 2 "https://github.com/TweetyDaBird")
+    (comment 3 "Licensed under Creative Commons BY-SA 4.0 International")
+  )
   (junction (at 92.71 106.68) (diameter 0) (color 0 0 0 0)
   )
@@
       (effects (font (size 1.27 1.27)) hide)
     )
+    (property "LCSC" "C588524" (at 120.65 177.8 0)
+      (effects (font (size 1.27 1.27)) hide)
+    )
