File: Rear Plate/Nearfield RP2040 RP.kicad_pcb (KiCad board)
At the start: 2 copper layers, 364.8 x 149.2 mm, 8 parts

Commit message: V1.00
Full design ready
Parts:
- added H10: Spacer_PCB, Keyboard_Plate:Spacer_Plate_Grounded_m3, F.Cu at (153.2, 81.2)
- added H9: Spacer_PCB, Keyboard_Plate:Spacer_Plate_Grounded_m3, F.Cu at (186.2, 81.2)
- added Logo1: CC-BY-SA-4.0, Logotypes:CC_BY_SA_40, F.Cu at (197.1, 185.2)
- H1, H2, H3, H4, H5, H6, H7, H8: footprint Keyboard_Plate:Spacer Plate hole -> Keyboard_Plate:Spacer_Plate_Grounded
Routing:
- added copper zone on B.Cu, net GND
- added copper zone on F.Cu, net GND
- removed copper zone on B.Cu, net (none)
- removed copper zone on F.Cu, net (none)
Other:
- board size 364.8 x 149.2 mm -> 364.8 x 148.8 mm
- board text added: "JLCJLCJLCJLC"
- board text added: "Royal Nearfield Rear - v1.00 Markus Knutsson 2024 https://github.com/TweetyDaBird"
